File: Diseño/Hardware/PCB/Final_1.kicad_pcb (KiCad board)
At the start: 2 copper layers, 105 x 85 mm, 147 parts, among them J1 Entrada transformador, J10 Conn_01x02_Male, J2 Conn_01x02_Male, J3 Conn_01x02_Male, J4 Conn_01x02_Male, J5 Conn_01x02_Male, J6 Conn_01x02_Male, J7 Entrada transformador, J8 Entrada transformador, J9 Conn_01x02_Male, Q1 BC848, U1 LM2575-5.0BU, U10 H11AA1, U11 H11AA1, U12 MOC3021M, U13 MOC3021M, U14 MOC3021M, U15 MOC3021M, U16 MOC3021M, U17 MOC3021M, U18 MOC3021M, U19 MOC3021M, U2 LM1117-3.3, U20 MOC3021M, U3 ESP-12F, U4 ATmega328-AU, U5 ACS712xLCTR-05B, U6 MOC3021M, U7 H11AA1, U8 H11AA1, U9 H11AA1, Y1 16Mhz

Commit message: Planos montaje
Routing:
- net Entrada_5: track 19.5 -> 24.7 mm
- net Entrada_4: track 14.1 -> 16.4 mm
- net GND: vias 4 -> 7
- net (no net): vias 0 -> 3
Changed lines of the file:
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@@
     (thickness 1.6)
     (drawings 6)
-    (tracks 792)
+    (tracks 801)
     (zones 0)
     (modules 147)
@@
   (layers
     (0 F.Cu signal)
-    (31 B.Cu signal hide)
+    (31 B.Cu signal)
     (32 B.Adhes user hide)
     (33 F.Adhes user hide)
@@
     (38 B.Mask user hide)
     (39 F.Mask user hide)
-    (40 Dwgs.User user hide)
+    (40 Dwgs.User user)
     (41 Cmts.User user hide)
     (42 Eco1.User user hide)
@@
     (via_min_size 0.4)
     (via_min_drill 0.3)
+    (user_via 3.5 3)
     (uvia_size 0.3)
     (uvia_drill 0.1)
@@
     )
   )
+  (dimension 85 (width 0.15) (layer Dwgs.User)
+    (gr_text "85,000 mm" (at 63.6 107.5 270) (layer Dwgs.User)
+      (effects (font (size 1 1) (thickness 0.15)))
+    )
+    (feature1 (pts (xy 70.75 150) (xy 64.313579 150)))
+    (feature2 (pts (xy 70.75 65) (xy 64.313579 65)))
+    (crossbar (pts (xy 64.9 65) (xy 64.9 150)))
+    (arrow1a (pts (xy 64.9 150) (xy 64.313579 148.873496)))
+    (arrow1b (pts (xy 64.9 150) (xy 65.486421 148.873496)))
+    (arrow2a (pts (xy 64.9 65) (xy 64.313579 66.126504)))
+    (arrow2b (pts (xy 64.9 65) (xy 65.486421 66.126504)))
+  )
+  (dimension 105 (width 0.15) (layer Dwgs.User)
+    (gr_text "105,000 mm" (at 123.25 58.100001) (layer Dwgs.User)
+      (effects (font (size 1 1) (thickness 0.15)))
+    )
+    (feature1 (pts (xy 70.75 65) (xy 70.75 58.81358)))
+    (feature2 (pts (xy 175.75 65) (xy 175.75 58.81358)))
+    (crossbar (pts (xy 175.75 59.400001) (xy 70.75 59.400001)))
+    (arrow1a (pts (xy 70.75 59.400001) (xy 71.876504 58.81358)))
+    (arrow1b (pts (xy 70.75 59.400001) (xy 71.876504 59.986422)))
+    (arrow2a (pts (xy 175.75 59.400001) (xy 174.623496 58.81358)))
+    (arrow2b (pts (xy 175.75 59.400001) (xy 174.623496 59.986422)))
+  )
   (gr_line (start 175.75 150) (end 175.75 65) (layer Edge.Cuts) (width 0.1))
   (gr_line (start 70.75 65) (end 175.75 65) (layer Edge.Cuts) (width 0.1))
-  (gr_line (start 60 152) (end 81 152) (layer Dwgs.User) (width 0.15))
-  (gr_line (start 60 145) (end 197 145) (layer Dwgs.User) (width 0.15))
   (gr_line (start 70.75 150) (end 70.75 65) (layer Edge.Cuts) (width 0.1))
   (gr_line (start 70.75 150) (end 175.75 150) (layer Edge.Cuts) (width 0.1))
+  (via (at 171 138) (size 3.5) (drill 3) (layers F.Cu B.Cu) (net 0))
+  (via (at 146 138) (size 3.5) (drill 3) (layers F.Cu B.Cu) (net 0))
+  (via (at 75 146) (size 3.5) (drill 3) (layers F.Cu B.Cu) (net 0))
   (segment (start 87.6625 111.5) (end 87.175 111.5) (width 0.3) (layer F.Cu) (net 1))
   (segment (start 83.5 89) (end 81.25 89) (width 0.3) (layer F.Cu) (net 1))
@@
   (segment (start 74.5625 125) (end 74.5625 119.6875) (width 0.3) (layer F.Cu) (net 4))
   (via (at 139.75 99.75) (size 0.8) (drill 0.4) (layers F.Cu B.Cu) (net 4))
+  (via (at 75 69) (size 3.5) (drill 3) (layers F.Cu B.Cu) (net 4))
+  (via (at 103 69) (size 3.5) (drill 3) (layers F.Cu B.Cu) (net 4))
+  (via (at 172 69) (size 3.5) (drill 3) (layers F.Cu B.Cu) (net 4))
   (segment (start 164.5 71.8125) (end 162.5 71.8125) (width 0.3) (layer F.Cu) (net 5))
   (segment (start 142 72.25) (end 142 77.25) (width 0.3) (layer F.Cu) (net 5))
@@
   (segment (start 161 127.5) (end 158.5625 127.5) (width 0.3) (layer F.Cu) (net 29))
   (segment (start 161 127.5) (end 161 144.5) (width 0.3) (layer B.Cu) (net 29))
-  (segment (start 168.5 131.4375) (end 168.5 134.5) (width 0.3) (layer B.Cu) (net 30))
-  (segment (start 168.5 134.5) (end 166 137) (width 0.3) (layer B.Cu) (net 30))
-  (segment (start 166 137) (end 166 144.5) (width 0.3) (layer B.Cu) (net 30))
+  (segment (start 168.5 131.4375) (end 165.0375 134.9) (width 0.3) (layer B.Cu) (net 30))
+  (segment (start 165.0375 144.9575) (end 166.08 146) (width 0.3) (layer B.Cu) (net 30))
+  (segment (start 165.0375 134.9) (end 165.0375 144.9575) (width 0.3) (layer B.Cu) (net 30))
   (segment (start 121.55 88.925) (end 121.625 89) (width 0.3) (layer F.Cu) (net 31))
   (segment (start 121.55 85.5) (end 121.55 88.925) (width 0.3) (layer F.Cu) (net 31))
@@
   (segment (start 171 127.5) (end 171 127.5) (width 0.3) (layer F.Cu) (net 86))
   (via (at 171 127.5) (size 0.8) (drill 0.4) (layers F.Cu B.Cu) (net 86))
-  (segment (start 171 127.5) (end 171 144.5) (width 0.3) (layer B.Cu) (net 86))
+  (segment (start 171 127.5) (end 171 131.7) (width 0.3) (layer B.Cu) (net 86))
+  (segment (start 171 131.7) (end 166.6 136.1) (width 0.3) (layer B.Cu) (net 86))
+  (segment (start 166.6 141.44) (end 171.16 146) (width 0.3) (layer B.Cu) (net 86))
+  (segment (start 166.6 136.1) (end 166.6 141.44) (width 0.3) (layer B.Cu) (net 86))
   (segment (start 113.54 128.11) (end 113.3 128.35) (width 0.25) (layer B.Cu) (net 87))
   (segment (start 113.54 123.31) (end 113.54 128.11) (width 0.25) (layer B.Cu) (net 87))

Commit message: Actualización pcb
Parts:
- added J11: SPI, Connector_PinSocket_2.54mm:PinSocket_2x03_P2.54mm_Vertical, F.Cu at (147.4, 81.5)
- J1: value Entrada transformador -> Entrada
- J2: value Conn_01x02_Male -> l
- J7: value Entrada transformador -> transformador
- J8: value Entrada transformador -> Salidas a relés
- R5: value 1,8 -> 1k8
- R6: value 3,3 -> 3k3
Connections:
- net Net-(R10-Pad2) renamed RST
Routing:
- net S6: track 17.5 -> 55.1 mm, vias 0 -> 1
- net S8: track 8.28 -> 37.3 mm, vias 0 -> 1
- net S7: track 10.9 -> 36.6 mm, vias 0 -> 1
- net RST: track 6.39 -> 18.9 mm, vias 0 -> 1
- net 5V: track 299.1 -> 309.4 mm
- net S1: track 60.0 -> 61.2 mm
- net S2: track 54.7 -> 55.5 mm
- net GND: vias 7 -> 8
