File: Diseño/Hardware/PCB/Final_1.sch (KiCad schematic (older format))
At the start: 147 parts, among them J1 Entrada transformador, J10 Conn_01x02_Male, J2 Conn_01x02_Male, J3 Conn_01x02_Male, J4 Conn_01x02_Male, J5 Conn_01x02_Male, J6 Conn_01x02_Male, J7 Entrada transformador, J8 Entrada transformador, J9 Conn_01x02_Male, Q1 BC848, U1 LM2575-5.0BU, U10 H11AA1, U11 H11AA1, U12 MOC3021M, U13 MOC3021M, U14 MOC3021M, U15 MOC3021M, U16 MOC3021M, U17 MOC3021M, U18 MOC3021M, U19 MOC3021M, U2 LM1117-3.3, U20 MOC3021M, U3 ESP-12F, U4 ATmega328-AU, U5 ACS712xLCTR-05B, U6 MOC3021M, U7 H11AA1, U8 H11AA1, U9 H11AA1, Y1 16Mhz

Commit message: Esquematicos y PCB
Parts:
- J1: value Entrada transformador -> Entrada
- J2: value Conn_01x02_Male -> l
- J7: value Entrada transformador -> transformador
- J8: value Entrada transformador -> Salidas a relés
- R5: value 1,8 -> 1k8
- R6: value 3,3 -> 3k3
Other:
- note added: "Entrada \nTransformador"
- note added: "Entrada\n sensores\ntemperatura"
- note added: "Entradas \npulsador"
- note added: "Salidas a relés"

Commit message: Actualización pcb
Parts:
- added J11: SPI, Connector_PinSocket_2.54mm:PinSocket_2x03_P2.54mm_Vertical, symbol Connector_Generic:Conn_02x03_Odd_Even
Connections:
- net 5V: now also J11.1 (Pin_1)
- net GND: now also J11.5 (Pin_5)
- net S6: now also J11.3 (Pin_3)
- net S7: now also J11.2 (Pin_2)
- net S8: now also J11.4 (Pin_4)
- net RST: now reaches R10.2, U4.29 (~RESET~/PC6)
- net RST: now also J11.6 (Pin_6)
Changed lines of the file:
@@
 	2200 6600 2250 6600
 Wire Wire Line
-	2200 5700 2700 5700
+	2200 5700 2600 5700
 Text GLabel 3350 5700 2    50   Input ~ 0
 5V
@@
 Text Notes 4400 5800 0    50   ~ 0
    Entrada \nTransformador
+$Comp
+L Connector_Generic:Conn_02x03_Odd_Even J11
+U 1 1 5F24108F
+P 7000 4350
+F 0 "J11" H 7050 4667 50  0000 C CNN
+F 1 "SPI" H 7050 4576 50  0000 C CNN
+F 2 "Connector_PinSocket_2.54mm:PinSocket_2x03_P2.54mm_Vertical" H 7000 4350 50  0001 C CNN
+F 3 "~" H 7000 4350 50  0001 C CNN
+	1    7000 4350
+	1    0    0    -1
+$EndComp
+Text GLabel 6800 4250 0    50   Input ~ 0
+5V
+$Comp
+L power:GND #PWR0101
+U 1 1 5F245110
+P 6800 4450
+F 0 "#PWR0101" H 6800 4200 50  0001 C CNN
+F 1 "GND" H 6805 4277 50  0000 C CNN
+F 2 "" H 6800 4450 50  0001 C CNN
+F 3 "" H 6800 4450 50  0001 C CNN
+	1    6800 4450
+	1    0    0    -1
+$EndComp
+Text GLabel 7300 4250 2    50   Input ~ 0
+S7
+Text GLabel 6800 4350 0    50   Input ~ 0
+S6
+Text GLabel 7300 4350 2    50   Input ~ 0
+S8
+Text GLabel 7300 4450 2    50   Input ~ 0
+RST
+Text GLabel 3350 5500 2    50   Input ~ 0
+RST
+Wire Wire Line
+	3350 5500 2600 5500
+Wire Wire Line
+	2600 5500 2600 5700
+Connection ~ 2600 5700
+Wire Wire Line
+	2600 5700 2700 5700
 $EndSCHEMATC
